File: Charlieplex84.sch (EAGLE design)
At the start: 115 parts, among them J1 ICSP

Commit message: update
Parts:
- U$3: value USER_HACKABLE -> (none); device logo:USER_HACKABLE -> 4h:4H-LOGO6
Changed lines of the file:
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@@
 <part name="S1" library="barbary_enterprises" deviceset="TAC_SWITCH" device="PTH"/>
 <part name="U$2" library="battery" deviceset="CR2032" device="THM"/>
-<part name="U$3" library="logo" deviceset="USER_HACKABLE" device=""/>
+<part name="U$3" library="4h" deviceset="4H-LOGO" device="6"/>
 </parts>
 <sheets>
@@
 <instance part="S1" gate="S" x="182.88" y="63.5"/>
 <instance part="U$2" gate="G$1" x="182.88" y="33.02" rot="R90"/>
-<instance part="U$3" gate="G$1" x="205.74" y="88.9"/>
+<instance part="U$3" gate="G$1" x="180.34" y="93.98"/>
 </instances>
 <busses>
